File: PCB/sch/Boros Rocket.kicad_sch (KiCad schematic)
At the start: 43 parts, among them J1 B2B-XH-A, J2 TYPE-C-31-M-12, J3 Conn_01x02_Pin, Q1 MMBT3904, U1 BMP390, U2 IAM-20381, U3 ICM-42688-P, U4 MCP73831T-2DCI_MC, U5 RP2040, U6 USBLC6-2SC6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

Commit message: Refactor code structure for improved readability and maintainability
Parts:
- removed C10, C9: 100 nF, Capacitor_SMD:C_0603_1608Metric, symbol Device:C
- removed C11, C19: 1µF, Capacitor_SMD:C_0603_1608Metric, symbol Device:C
- removed C17, C18: 22pF, Capacitor_SMD:C_0603_1608Metric, symbol Device:C
- removed C20, C7, C8: 100nF, Capacitor_SMD:C_0603_1608Metric, symbol Device:C
- removed J2: TYPE-C-31-M-12, OPL:HRO_TYPE-C-31-M-12, symbol TYPE-C-31-M-12:TYPE-C-31-M-12
- removed J3: Conn_01x02_Pin, Connector_PinHeader_2.54mm:PinHeader_1x02_P2.54mm_Vertical, symbol Connector:Conn_01x02_Pin
- removed R5: 22Ω, Resistor_SMD:R_0603_1608Metric, symbol Device:R
- removed R7: 10k, Resistor_SMD:R_0603_1608Metric, symbol Device:R
- removed U2: IAM-20381, OPL:PQFN50P300X300X80-16N, symbol IAM-20381:IAM-20381
- removed U5: RP2040, OPL:QFN40P700X700X90-57N, symbol RP2040:RP2040
- removed U8: W25Q32JVSSIQ, OPL:SOIC127P790X216-8N, symbol W25Q32JVSSIQ:W25Q32JVSSIQ
- removed Y1: 12MHz, Crystal:Crystal_SMD_3225-4Pin_3.2x2.5mm, symbol Device:Crystal
- added J2: 1981568-1, OPL:TE_1981568-1, symbol 1981568-1:1981568-1
- added J4: Conn_02x04_Counter_Clockwise, Connector_PinHeader_2.54mm:PinHeader_2x04_P2.54mm_Vertical, symbol Connector_Generic:Conn_02x04_Counter_Clockwise
- added U2: STM32G071K8TxN, Package_QFP:LQFP-32_7x7mm_P0.8mm, symbol MCU_ST_STM32G0:STM32G071K8TxN
- R1, R2: value 5.1 kΩ -> 100k
- R4: value 22Ω -> 10k
Connections:
- net BARO_CS: now also U2.16 (PB1)
- net BUZZER_EN: now also U2.1 (PB9)
- net CHG_STAT: now also U2.3 (PC15)
- net FLASH_CS: now also U2.11 (PA4)
- net GND: now also C5.1, R2.2, J2.5, J2.SH1 (SHIELD), J2.SH2 (SHIELD), J2.SH3 (SHIELD), J2.SH4 (SHIELD), J2.SH5 (SHIELD), J2.SH6 (SHIELD), J4.8 (Pin_8), U2.5 (VSS); no longer C5.2, R1.1, R2.1
- net IMU_CS: now also U2.15 (PB0)
- net IMU_INT1: now also U2.30 (PB6)
- net IMU_INT2: now also U2.31 (PB7)
- net SPI_MISO: now also U2.13 (PA6)
- net SPI_MOSI: now also U2.14 (PA7)
- net SPI_SCK: now also U2.12 (PA5)
- net USB_DM: now also J2.2, U2.22 (PA9/PA11)
- net USB_DP: now also J2.3, U2.23 (PA10/PA12); no longer R4.1
- net USB_VBUS: now reaches R1.2
- net USB_VBUS: now also J2.1, J4.5 (Pin_5)
- net NRST: now reaches R4.2
- net NRST: now also C6.1, J4.1 (Pin_1), U2.6 (PF2)
- net BARO_INT: no longer names the net of U1.INT
- net DVDD renamed 3V3
- net 3V3: now also R4.1, J4.4 (Pin_4), U2.4 (VDD); no longer C5.1, C6.1
- new net SWCLK: J4.3 (Pin_3), U2.25 (PA14)
- new net SWDIO: J4.2 (Pin_2), U2.24 (PA13)
- new net UART_RX: J4.6 (Pin_6), U2.10 (PA3)
- new net UART_TX: J4.7 (Pin_7), U2.9 (PA2)
- new net USB_VBUS_SENSE: C5.2, R1.1, R2.1, U2.18 (PA8)
- no-connect marks 27 -> 19
